Commit message: 0729(ChatGPT navigation and camera)

File: turtlebot3/turtlebot3/turtlebot3_description/urdf/turtlebot3_burger.gazebo.xacro (robot description, xacro)
@@ -3,7 +3,36 @@
   <xacro:arg name="laser_visual" default="false"/>
   <xacro:arg name="imu_visual"   default="false"/>
+    <!-- jylong start -->
+  <xacro:include filename="$(find realsense2_description)/urdf/_d435.urdf.xacro" />
+  <!-- jylong end -->
+  <!-- jylong start-->
+  <xacro:sensor_d435 name="camera" topics_ns="camera" parent="base_link" publish_pointcloud="true">
+    <origin xyz="0 0 0.1" rpy="0 0 0" />
+  </xacro:sensor_d435>
+ <!-- jylong end-->
   <gazebo reference="base_link">
     <material>Gazebo/DarkGrey</material>
   </gazebo>
+  <!-- jylong start-->
+  <gazebo reference="camera_link">
+    <gravity>true</gravity>
+    <sensor name="imu_sensor" type="imu">
+      <always_on>true</always_on>
+      <update_rate>200</update_rate>
+      <visualize>true</visualize>
+      <topic>__default_topic__</topic>
+      <plugin filename="libgazebo_ros_imu_sensor.so" name="imu_plugin">
+        <topicName>d435i/imu</topicName>
+        <bodyName>camera_link</bodyName>
+        <updateRateHZ>200.0</updateRateHZ>
+        <gaussianNoise>0.0</gaussianNoise>
+        <xyzOffset>0.0 0.0 0.0</xyzOffset>
+        <rpyOffset>0.0 0.0 0.0</rpyOffset>
+        <frameName>imu_link_</frameName>
+      </plugin>
+      <pose>0 0 0 0 0 0</pose>
+    </sensor>
+  </gazebo>
+ <!-- jylong end-->
   <gazebo reference="wheel_left_link">
     <mu1>0.1</mu1>
